Commit message: Version working with CustomControl - Only pose command

File: kimm_description/urdf/kimm_stewart_platform.xacro (robot description, xacro)
@@ -33,4 +33,5 @@
     <link name="platform_roll"/>
     <link name="platform_pitch"/>
+    <link name="platform_yaw"/>
     <link name="distal_ring">
       <visual>
@@ -68,9 +69,5 @@
     <!--
       Translation Z.
-      The joint origin defines the nominal/home height of the distal platform.
-      The joint value then represents displacement relative to this home pose.
-      Example:
-        platform_z_joint = 0.0  -> distal ring at z = 0.131 m
-        platform_z_joint = 0.019 -> distal ring at z = 0.15 m
+      The joint value represents displacement relative to this home pose.
     -->
     <joint name="platform_z_joint" type="prismatic">
@@ -100,8 +97,14 @@
     <joint name="platform_yaw_joint" type="revolute">
       <parent link="platform_pitch"/>
-      <child link="distal_ring"/>
+      <child link="platform_yaw"/>
       <origin xyz="0 0 0" rpy="0 0 0"/>
       <axis xyz="0 0 1"/>
       <limit lower="-3.14" upper="3.14" effort="100" velocity="1.0"/>
+    </joint>
+    <!-- Attach distal ring mesh to the final virtual yaw frame -->
+    <joint name="platform_yaw_to_distal_ring" type="fixed">
+      <parent link="platform_yaw"/>
+      <child link="distal_ring"/>
+      <origin xyz="0 0 0" rpy="0 0 0"/>
     </joint>
     <!-- Tool/probe guide frame attached to the moving platform -->

Commit message: Hardware working version

File: kimm_description/urdf/kimm_stewart_platform.xacro (robot description, xacro)
@@ -8,5 +8,5 @@
     <link name="proximal_ring">
       <visual>
-        <origin xyz="0.035 -0.125 0" rpy="0 0 1.0471975511965976"/>
+        <origin xyz="0.035 -0.125 -0.133" rpy="0 0 1.0471975511965976"/>
         <geometry>
           <mesh filename="package://kimm_description/meshes/visual/base_plate.stl"
@@ -16,5 +16,5 @@
       </visual>
       <collision>
-        <origin xyz="0.035 -0.125 0" rpy="0 0 1.0471975511965976"/>
+        <origin xyz="0.035 -0.125 -0.133" rpy="0 0 1.0471975511965976"/>
         <geometry>
           <mesh filename="package://kimm_description/meshes/visual/base_plate.stl"
@@ -36,5 +36,5 @@
     <link name="distal_ring">
       <visual>
-        <origin xyz="-0.0815 0.022 0.131" rpy="0 0 -1.0471975511965976"/>
+        <origin xyz="-0.0815 0.022 0" rpy="0 0 -1.0471975511965976"/>
         <geometry>
           <mesh filename="package://kimm_description/meshes/visual/top_plate.stl"
@@ -44,5 +44,5 @@
       </visual>
       <collision>
-        <origin xyz="-0.0815 0.022 0.131" rpy="0 0 -1.0471975511965976"/>
+        <origin xyz="-0.0815 0.022 0" rpy="0 0 -1.0471975511965976"/>
         <geometry>
           <mesh filename="package://kimm_description/meshes/visual/top_plate.stl"
